File: Definitivi/uNav44_r1.sch (EAGLE design)
At the start: 37 parts, among them IC1 DSPIC33FJ128MC, IC2 24LC024, Q1 10MHz

Commit message: Add Vencoder voltage selection \ Removed connection of LED3 and LED4 from connector \ @katodo : PCB update is needed
Parts:
- removed SJ1, SJ2: (no value), jumper:SJ
- added SJ3: (no value), jumper:SJ2W
Connections:
- removed net VENC1: SJ2.2, SV1.3
- removed net VENC2: SJ1.2, SV1.4
- new net VENC: SV1.3, SV1.4
- net +3V3: now also SJ3.1
- net +5V: now also SJ3.3
- net VENC1-LD3: no longer SJ2.1
- net VENC2-LD4: no longer SJ1.1
Other:
- note added: "IO7 and IO8 can be used as Z channel of encoder"
- note removed: "Optionnaly, without LED monted, we can use VENC1/VENC2 input as Z channel of encoder"
