File: Definitivi/uBridge44_r1.sch (EAGLE design)
At the start: 18 parts

Commit message: encoder connettor for motor / @katodo ready for you
Parts:
- added JP1, JP2: (no value), pinhead:PINHD-2X2
Connections:
- removed net VENC1: SV2.3
- removed net VENC2: SV2.4
- new net VENC: JP1.3, JP2.3, SV2.3, SV2.4
- net CHA1: now also JP2.2
- net CHA2: now also JP1.2
- net CHB1: now also JP2.4
- net CHB2: now also JP1.4
- net GND: now also JP1.1, JP2.1
