File: Design/uNav44_r1.sch (EAGLE design)
At the start: 73 parts, among them IC1 DSPIC33FJ128MC, IC2 24LC024, IC3 AP3417CK-3.3TRG1, IC4 AP6503SP-13, U1 MCP6G01T-E/OT, U2 MCP6G01T-E/OT, U3 MCP6G01T-E/OT, U4 MCP6G01T-E/OT

Commit message: First release with 100% routing complete... and some error :)
Parts:
- added H4: MOUNT-PAD-ROUND2.8, holes:MOUNT-PAD-ROUND2.8
Connections:
- removed net IO0: SV2.12
- net GND: now also H4.MOUNT
- net IO3: now also SV2.12; no longer SV2.18
Changed lines of the file:
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@@
 <part name="JP4" library="OfficineRobotiche" deviceset="0R-JUMP-4" device=""/>
 <part name="JP5" library="OfficineRobotiche" deviceset="0R-JUMP-4" device=""/>
+<part name="H4" library="holes" deviceset="MOUNT-PAD-ROUND" device="2.8"/>
+<part name="GND37" library="supply1" deviceset="GND" device=""/>
 </parts>
 <sheets>
@@
 </segment>
 <segment>
-<wire x1="60.96" y1="12.7" x2="55.88" y2="12.7" width="0.1524" layer="91"/>
-<label x="55.88" y="12.7" size="0.8128" layer="95" font="vector" rot="MR0" xref="yes"/>
-<pinref part="SV2" gate="G$1" pin="18"/>
-</segment>
-<segment>
 <wire x1="106.68" y1="48.26" x2="104.14" y2="48.26" width="0.1524" layer="91"/>
 <label x="104.14" y="48.26" size="0.8128" layer="95" font="vector" ratio="13" rot="R180" xref="yes"/>
 <pinref part="JP4" gate="-0R" pin="4"/>
 </segment>
+<segment>
+<wire x1="60.96" y1="20.32" x2="55.88" y2="20.32" width="0.1524" layer="91"/>
+<label x="55.88" y="20.32" size="0.8128" layer="95" font="vector" rot="MR0" xref="yes"/>
+<pinref part="SV2" gate="G$1" pin="12"/>
+</segment>
 </net>
 <net name="IO2" class="0">
@@
 <net name="IO0" class="0">
 <segment>
-<wire x1="60.96" y1="20.32" x2="55.88" y2="20.32" width="0.1524" layer="91"/>
-<label x="55.88" y="20.32" size="0.8128" layer="95" font="vector" rot="MR0" xref="yes"/>
-<pinref part="SV2" gate="G$1" pin="12"/>
+<wire x1="55.88" y1="5.08" x2="50.8" y2="5.08" width="0.1524" layer="91"/>
+<label x="50.8" y="5.08" size="0.8128" layer="95" font="vector" rot="MR0" xref="yes"/>
 </segment>
 </net>
@@
 <pinref part="+3V5" gate="G$1" pin="+3V3"/>
 <wire x1="73.66" y1="40.64" x2="73.66" y2="38.1" width="0.1524" layer="91"/>
-<wire x1="76.2" y1="30.48" x2="78.74" y2="30.48" width="0.1524" layer="91"/>
 <label x="81.28" y="30.48" size="0.8128" layer="95" font="vector" rot="MR180" xref="yes"/>
 <wire x1="78.74" y1="30.48" x2="81.28" y2="30.48" width="0.1524" layer="91"/>
 <wire x1="73.66" y1="38.1" x2="78.74" y2="38.1" width="0.1524" layer="91"/>
 <wire x1="78.74" y1="38.1" x2="78.74" y2="30.48" width="0.1524" layer="91"/>
+<wire x1="78.74" y1="30.48" x2="76.2" y2="30.48" width="0.1524" layer="91"/>
+<pinref part="SV2" gate="G$1" pin="3"/>
 <junction x="78.74" y="30.48"/>
-<pinref part="SV2" gate="G$1" pin="3"/>
 </segment>
 <segment>
@@
 <attribute name="VALUE" x="139.7" y="55.88" size="1.27" layer="96"/>
 </instance>
+<instance part="H4" gate="G$1" x="210.82" y="93.98" smashed="yes" rot="R90">
+<attribute name="NAME" x="210.2358" y="96.774" size="1.27" layer="95" rot="R90"/>
+<attribute name="VALUE" x="213.2838" y="96.774" size="1.27" layer="96" rot="R90"/>
+</instance>
+<instance part="GND37" gate="1" x="210.82" y="86.36" smashed="yes">
+<attribute name="VALUE" x="213.36" y="85.09" size="1.27" layer="96" rot="R180"/>
+</instance>
 </instances>
 <busses>
@@
 <wire x1="142.24" y1="60.96" x2="142.24" y2="66.04" width="0.1524" layer="91"/>
 </segment>
-</net>
+<segment>
+<pinref part="H4" gate="G$1" pin="MOUNT"/>
+<pinref part="GND37" gate="1" pin="GND"/>
+<wire x1="210.82" y1="88.9" x2="210.82" y2="91.44" width="0.1524" layer="91"/>
+</segment>
+</net>

Commit message: Update of some file
Parts:
- SV1, SV2: device con-lstb:MA10-2 -> OfficineRobotiche:MA10-2
Connections:
- net IO3: now also SV2.18; no longer SV2.12
Changed lines of the file:
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@@
 </variantdefs>
 <classes>
-<class number="0" name="default" width="0.254" drill="0.4064">
-<clearance class="0" value="0.1778"/>
+<class number="0" name="default" width="0.254" drill="0.3048">
+<clearance class="0" value="0.2032"/>
 </class>
-<class number="1" name="power" width="0.3048" drill="0.4064">
+<class number="1" name="power" width="0.254" drill="0.3048">
 <clearance class="1" value="0.2032"/>
 </class>
@@
 <part name="P+5" library="supply1" deviceset="+12V" device=""/>
 <part name="GND12" library="supply1" deviceset="GND" device=""/>
-<part name="SV2" library="con-lstb" deviceset="MA10-2" device=""/>
-<part name="SV1" library="con-lstb" deviceset="MA10-2" device="">
+<part name="SV2" library="OfficineRobotiche" deviceset="MA10-2" device=""/>
+<part name="SV1" library="OfficineRobotiche" deviceset="MA10-2" device="">
 <attribute name="MF" value=""/>
 <attribute name="MPN" value=""/>
@@
 </segment>
 <segment>
-<wire x1="60.96" y1="20.32" x2="55.88" y2="20.32" width="0.1524" layer="91"/>
-<label x="55.88" y="20.32" size="0.8128" layer="95" font="vector" rot="MR0" xref="yes"/>
-<pinref part="SV2" gate="G$1" pin="12"/>
+<label x="55.88" y="12.7" size="0.8128" layer="95" font="vector" rot="MR0" xref="yes"/>
+<pinref part="SV2" gate="G$1" pin="18"/>
+<wire x1="55.88" y1="12.7" x2="60.96" y2="12.7" width="0.1524" layer="91"/>
 </segment>
 </net>
@@
 </segment>
 </net>
-<net name="IO0" class="0">
-<segment>
-<wire x1="55.88" y1="5.08" x2="50.8" y2="5.08" width="0.1524" layer="91"/>
-<label x="50.8" y="5.08" size="0.8128" layer="95" font="vector" rot="MR0" xref="yes"/>
-</segment>
-</net>
