File: Design/uNav44_r1.sch (EAGLE design)
At the start: 74 parts, among them IC1 DSPIC33FJ128MC, IC2 24LC024, IC3 AP3417CK-3.3TRG1, IC4 AP6503SP-13, U1 MCP6G01T-E/OT, U2 MCP6G01T-E/OT, U3 MCP6G01T-E/OT, U4 MCP6G01T-E/OT

Commit message: uNAV44 finished.
Parts:
- removed TP3, TP4, TP5: PTR1TP07R, testpad:PTR1TP07R
- JP1: value M02LOCK -> M02PTH; device SparkFun-Connectors:M02LOCK -> SparkFun-Connectors:M02PTH
- renumbered JMP5 to J6, JMP6 to J7, JP2 to J2, JP3 to J3, JP4 to J4, JP5 to J5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
Connections:
- removed net HALT: IC1.TDI/PMA9/RA9
- new net IO0: IC1.TDI/PMA9/RA9, SV2.12
